Commit message: completed

File: BadBot_description/urdf/BadBot.xacro (robot description, xacro)
@@ -8,7 +8,7 @@
 <link name="base_link">
   <inertial>
-    <origin xyz="-0.016271579372150194 0.14227699615361108 0.13718460738785923" rpy="0 0 0"/>
-    <mass value="28.94724121287408"/>
-    <inertia ixx="0.483788" iyy="0.452084" izz="0.900633" ixy="0.0" iyz="-0.002009" ixz="0.0"/>
+    <origin xyz="-0.016271579372150208 0.1417094158489788 0.1370115013532809" rpy="0 0 0"/>
+    <mass value="28.855052709016757"/>
+    <inertia ixx="0.480495" iyy="0.451805" izz="0.897614" ixy="0.0" iyz="-0.001119" ixz="0.0"/>
   </inertial>
   <visual>
@@ -26,5 +26,5 @@
   </collision>
 </link>
-<link name="caster_wheel_1_1_1">
+<link name="caster_wheel_1">
   <inertial>
     <origin xyz="4.2062784975580025e-07 1.9035339363093762e-07 -1.0802124120190548e-07" rpy="0 0 0"/>
@@ -35,5 +35,5 @@
     <origin xyz="0.016272 -0.029802 -0.093867" rpy="0 0 0"/>
     <geometry>
-      <mesh filename="package://BadBot_description/meshes/caster_wheel_1_1_1.stl" scale="0.001 0.001 0.001"/>
+      <mesh filename="package://BadBot_description/meshes/caster_wheel_1.stl" scale="0.001 0.001 0.001"/>
     </geometry>
     <material name="silver"/>
@@ -42,9 +42,9 @@
     <origin xyz="0.016272 -0.029802 -0.093867" rpy="0 0 0"/>
     <geometry>
-      <mesh filename="package://BadBot_description/meshes/caster_wheel_1_1_1.stl" scale="0.001 0.001 0.001"/>
+      <mesh filename="package://BadBot_description/meshes/caster_wheel_1.stl" scale="0.001 0.001 0.001"/>
     </geometry>
   </collision>
 </link>
-<link name="right_wheel_2_1_1">
+<link name="right_wheel_1">
   <inertial>
     <origin xyz="4.206278496621252e-07 -1.21080121928685e-07 -1.0802128527775956e-07" rpy="0 0 0"/>
@@ -55,5 +55,5 @@
     <origin xyz="-0.133728 -0.221391 -0.108867" rpy="0 0 0"/>
     <geometry>
-      <mesh filename="package://BadBot_description/meshes/right_wheel_2_1_1.stl" scale="0.001 0.001 0.001"/>
+      <mesh filename="package://BadBot_description/meshes/right_wheel_1.stl" scale="0.001 0.001 0.001"/>
     </geometry>
     <material name="silver"/>
@@ -62,9 +62,29 @@
     <origin xyz="-0.133728 -0.221391 -0.108867" rpy="0 0 0"/>
     <geometry>
-      <mesh filename="package://BadBot_description/meshes/right_wheel_2_1_1.stl" scale="0.001 0.001 0.001"/>
+      <mesh filename="package://BadBot_description/meshes/right_wheel_1.stl" scale="0.001 0.001 0.001"/>
     </geometry>
   </collision>
 </link>
-<link name="left_wheel_1_1_1">
+<link name="right_wheel_axle_1">
+  <inertial>
+    <origin xyz="-0.04749957937215024 -1.2108012187317385e-07 -1.080212411880277e-07" rpy="0 0 0"/>
+    <mass value="0.23876104167282425"/>
+    <inertia ixx="1.2e-05" iyy="0.000186" izz="0.000186" ixy="0.0" iyz="-0.0" ixz="0.0"/>
+  </inertial>
+  <visual>
+    <origin xyz="-0.181228 -0.221391 -0.108867" rpy="0 0 0"/>
+    <geometry>
+      <mesh filename="package://BadBot_description/meshes/right_wheel_axle_1.stl" scale="0.001 0.001 0.001"/>
+    </geometry>
+    <material name="silver"/>
+  </visual>
+  <collision>
+    <origin xyz="-0.181228 -0.221391 -0.108867" rpy="0 0 0"/>
+    <geometry>
+      <mesh filename="package://BadBot_description/meshes/right_wheel_axle_1.stl" scale="0.001 0.001 0.001"/>
+    </geometry>
+  </collision>
+</link>
+<link name="left_wheel_1">
   <inertial>
     <origin xyz="4.2062784980090306e-07 -1.2108012190092943e-07 -1.0802128526388177e-07" rpy="0 0 0"/>
@@ -75,5 +95,5 @@
     <origin xyz="0.166272 -0.221391 -0.108867" rpy="0 0 0"/>
     <geometry>
-      <mesh filename="package://BadBot_description/meshes/left_wheel_1_1_1.stl" scale="0.001 0.001 0.001"/>
+      <mesh filename="package://BadBot_description/meshes/left_wheel_1.stl" scale="0.001 0.001 0.001"/>
     </geometry>
     <material name="silver"/>
@@ -82,74 +102,80 @@
     <origin xyz="0.166272 -0.221391 -0.108867" rpy="0 0 0"/>
     <geometry>
-      <mesh filename="package://BadBot_description/meshes/left_wheel_1_1_1.stl" scale="0.001 0.001 0.001"/>
+      <mesh filename="package://BadBot_description/meshes/left_wheel_1.stl" scale="0.001 0.001 0.001"/>
     </geometry>
   </collision>
 </link>
-<link name="r_wheel_shaft_2_1_1">
+<link name="_left_wheel_axle_1">
   <inertial>
-    <origin xyz="-0.04749957937215024 -1.2108012187317385e-07 -1.080212411880277e-07" rpy="0 0 0"/>
-    <mass value="0.23876104167282425"/>
+    <origin xyz="-0.04749957937215003 -1.2108012209521846e-07 -1.0802124131292778e-07" rpy="0 0 0"/>
+    <mass value="0.23876104167282444"/>
     <inertia ixx="1.2e-05" iyy="0.000186" izz="0.000186" ixy="0.0" iyz="-0.0" ixz="0.0"/>
   </inertial>
   <visual>
-    <origin xyz="-0.181228 -0.221391 -0.108867" rpy="0 0 0"/>
+    <origin xyz="0.118772 -0.221391 -0.108867" rpy="0 0 0"/>
     <geometry>
-      <mesh filename="package://BadBot_description/meshes/r_wheel_shaft_2_1_1.stl" scale="0.001 0.001 0.001"/>
+      <mesh filename="package://BadBot_description/meshes/_left_wheel_axle_1.stl" scale="0.001 0.001 0.001"/>
     </geometry>
     <material name="silver"/>
   </visual>
   <collision>
-    <origin xyz="-0.181228 -0.221391 -0.108867" rpy="0 0 0"/>
+    <origin xyz="0.118772 -0.221391 -0.108867" rpy="0 0 0"/>
     <geometry>
-      <mesh filename="package://BadBot_description/meshes/r_wheel_shaft_2_1_1.stl" scale="0.001 0.001 0.001"/>
+      <mesh filename="package://BadBot_description/meshes/_left_wheel_axle_1.stl" scale="0.001 0.001 0.001"/>
     </geometry>
   </collision>
 </link>
-<link name="l_wheel_shaft_1_1_1">
+<link name="lidar_v1_1">
   <inertial>
-    <origin xyz="0.047500420627849954 -1.2108012209521846e-07 -1.0802124131292778e-07" rpy="0 0 0"/>
-    <mass value="0.23876104167282444"/>
-    <inertia ixx="1.2e-05" iyy="0.000186" izz="0.000186" ixy="0.0" iyz="-0.0" ixz="0.0"/>
+    <origin xyz="-0.004865441389214329 0.1410900178145767 0.016766645484714182" rpy="0 0 0"/>
+    <mass value="0.3543299620873657"/>
+    <inertia ixx="0.000474" iyy="0.000229" izz="0.000616" ixy="-2.3e-05" iyz="3.1e-05" ixz="3e-06"/>
   </inertial>
   <visual>
-    <origin xyz="0.213772 -0.221391 -0.108867" rpy="0 0 0"/>
+    <origin xyz="0.016272 -0.146391 -0.178867" rpy="0 0 0"/>
     <geometry>
-      <mesh filename="package://BadBot_description/meshes/l_wheel_shaft_1_1_1.stl" scale="0.001 0.001 0.001"/>
+      <mesh filename="package://BadBot_description/meshes/lidar_v1_1.stl" scale="0.001 0.001 0.001"/>
     </geometry>
     <material name="silver"/>
   </visual>
   <collision>
-    <origin xyz="0.213772 -0.221391 -0.108867" rpy="0 0 0"/>
+    <origin xyz="0.016272 -0.146391 -0.178867" rpy="0 0 0"/>
     <geometry>
-      <mesh filename="package://BadBot_description/meshes/l_wheel_shaft_1_1_1.stl" scale="0.001 0.001 0.001"/>
+      <mesh filename="package://BadBot_description/meshes/lidar_v1_1.stl" scale="0.001 0.001 0.001"/>
     </geometry>
   </collision>
 </link>
-<joint name="Rigid12" type="fixed">
+<joint name="Rev7" type="continuous">
   <origin xyz="-0.016272 0.029802 0.093867" rpy="0 0 0"/>
   <parent link="base_link"/>
-  <child link="caster_wheel_1_1_1"/>
+  <child link="caster_wheel_1"/>
+  <axis xyz="0.0 0.0 -1.0"/>
 </joint>
-<joint name="Rev13" type="continuous">
+<joint name="Rev8" type="continuous">
   <origin xyz="-0.0475 0.0 0.0" rpy="0 0 0"/>
-  <parent link="r_wheel_shaft_2_1_1"/>
-  <child link="right_wheel_2_1_1"/>
+  <parent link="right_wheel_axle_1"/>
+  <child link="right_wheel_1"/>
   <axis xyz="-1.0 0.0 0.0"/>
 </joint>
-<joint name="Rev14" type="continuous">
-  <origin xyz="0.0475 0.0 0.0" rpy="0 0 0"/>
-  <parent link="l_wheel_shaft_1_1_1"/>
-  <child link="left_wheel_1_1_1"/>
+<joint name="Rigid9" type="fixed">
+  <origin xyz="0.181228 0.221391 0.108867" rpy="0 0 0"/>
+  <parent link="base_link"/>
+  <child link="right_wheel_axle_1"/>
+</joint>
+<joint name="Rev10" type="continuous">
+  <origin xyz="-0.0475 0.0 0.0" rpy="0 0 0"/>
+  <parent link="_left_wheel_axle_1"/>
+  <child link="left_wheel_1"/>
   <axis xyz="-1.0 0.0 0.0"/>
 </joint>
-<joint name="Rigid15" type="fixed">
-  <origin xyz="0.181228 0.221391 0.108867" rpy="0 0 0"/>
+<joint name="Rigid11" type="fixed">
+  <origin xyz="-0.118772 0.221391 0.108867" rpy="0 0 0"/>
   <parent link="base_link"/>
-  <child link="r_wheel_shaft_2_1_1"/>
+  <child link="_left_wheel_axle_1"/>
 </joint>
-<joint name="Rigid16" type="fixed">
-  <origin xyz="-0.213772 0.221391 0.108867" rpy="0 0 0"/>
+<joint name="Rigid12" type="fixed">
+  <origin xyz="-0.016272 0.146391 0.178867" rpy="0 0 0"/>
   <parent link="base_link"/>
-  <child link="l_wheel_shaft_1_1_1"/>
+  <child link="lidar_v1_1"/>
 </joint>
 </robot>
