Commit message: commented rviz node temporarily

File: BadBot_description/urdf/BadBot_old.urdf (robot description, URDF)
Before this commit: robot BadBot, 7 links, 6 joints
Links:
- link base_link: geometry collision mesh filename=file:///home/mayank/BadBot/BadBot_ros2_ws/install/BadBot_de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 scale=0.001 0.001 0.001; visual mesh filename=file:///home/mayank/BadBot/BadBot_ros2_ws/install/BadBot_de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 scale=0.001 0.001 0.001
- link caster_wheel_1: geometry collision mesh filename=file:///home/mayank/BadBot/BadBot_ros2_ws/install/BadBot_de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 scale=0.001 0.001 0.001; visual mesh filename=file:///home/mayank/BadBot/BadBot_ros2_ws/install/BadBot_de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 scale=0.001 0.001 0.001
- link left_shaft_1: geometry collision mesh filename=file:///home/mayank/BadBot/BadBot_ros2_ws/install/BadBot_de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 scale=0.001 0.001 0.001; visual mesh filename=file:///home/mayank/BadBot/BadBot_ros2_ws/install/BadBot_de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 scale=0.001 0.001 0.001
- link left_wheel_1: geometry collision mesh filename=file:///home/mayank/BadBot/BadBot_ros2_ws/install/BadBot_de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 scale=0.001 0.001 0.001; visual mesh filename=file:///home/mayank/BadBot/BadBot_ros2_ws/install/BadBot_de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 scale=0.001 0.001 0.001
- link lidar_1: geometry collision mesh filename=file:///home/mayank/BadBot/BadBot_ros2_ws/install/BadBot_de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 scale=0.001 0.001 0.001; visual mesh filename=file:///home/mayank/BadBot/BadBot_ros2_ws/install/BadBot_de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 scale=0.001 0.001 0.001
- link right_shaft_1: geometry collision mesh filename=file:///home/mayank/BadBot/BadBot_ros2_ws/install/BadBot_de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 scale=0.001 0.001 0.001; visual mesh filename=file:///home/mayank/BadBot/BadBot_ros2_ws/install/BadBot_de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 scale=0.001 0.001 0.001
- link right_wheel_1: geometry collision mesh filename=file:///home/mayank/BadBot/BadBot_ros2_ws/install/BadBot_de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 scale=0.001 0.001 0.001; visual mesh filename=file:///home/mayank/BadBot/BadBot_ros2_ws/install/BadBot_de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 scale=0.001 0.001 0.001
Joints:
- joint Rev10: type continuous -> revolute
- joint Rev7: type continuous -> ball
- joint Rev8: type continuous -> revolute

File: BadBot_description/urdf/BadBot_unarranged.urdf (robot description, URDF)
Before this commit: robot BadBot, 7 links, 6 joints
Joints:
- joint Rev7: axis (none) -> -0.0 -0.0 -1.0; type fixed -> continuous
